File: EnvSensorNode.kicad_pcb (KiCad board)
At the start: 4 copper layers, 50 x 30 mm, 44 parts, among them IC1 STM32L010C6T6, J1 Borad_Conn, J2 Conn_DBG, Q1 BSN20, Q2 BSN20, SW1 SW_RST, U1 BME280, U2 TS5A3159ADCKR, U3 TS5A3159ADCKR, U4 MCP6002-xMS, Y1 32.768k

Commit message: Make top gnd plane
Routing:
- added copper zone on F.Cu, net GND
- removed copper zone on F.Cu, net (none)
Changed lines of the file:
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@@
   (segment (start 125 67) (end 125.4425 67) (width 0.1) (layer "F.Cu") (net 51))
   (segment (start 125.4425 67) (end 125.8425 66.6) (width 0.1) (layer "F.Cu") (net 51))
-  (zone (net 0) (net_name "") (layer "F.Cu") (hatch edge 0.5)
+  (zone (net 1) (net_name "GND") (layer "F.Cu") (hatch edge 0.5)
     (connect_pads (clearance 0.5))
     (min_thickness 0.25) (filled_areas_thickness no)
